File: KiCAD/euro2breadboard v1.1/euro2breadboard.kicad_pcb (KiCad board)
At the start: 2 copper layers, 31.8 x 50.3 mm, 13 parts, among them J1 JST_BUS, J2 IDC_BUS, SW1 SW_DPDT_x2

Commit message: Added gerber files
Routing:
- net GND: vias 14 -> 47
- net (no net): vias 0 -> 2
Changed lines of the file:
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@@
     (thickness 1.6)
     (drawings 29)
-    (tracks 75)
+    (tracks 107)
     (zones 0)
     (modules 13)
@@
   (page A4)
   (layers
-    (0 F.Cu signal hide)
-    (31 B.Cu signal hide)
+    (0 F.Cu signal)
+    (31 B.Cu signal)
     (32 B.Adhes user)
     (33 F.Adhes user)
@@
       (drillshape 0)
       (scaleselection 1)
-      (outputdirectory "../../Fabrication/euro2breadboard v1.0/"))
+      (outputdirectory "../../Fabrication/euro2breadboard v1.1/"))
   )
   (net 0 "")
@@
     (arrow2b (pts (xy 61.087 43.815) (xy 61.673421 44.941504)))
   )
+  (via (at 85.1535 62.611) (size 0.8) (drill 0.4) (layers F.Cu B.Cu) (net 0))
+  (via (at 84.201 62.5475) (size 0.8) (drill 0.4) (layers F.Cu B.Cu) (net 0))
   (via (at 90.17 81.026) (size 0.8) (drill 0.4) (layers F.Cu B.Cu) (net 1))
   (via (at 88.646 82.296) (size 0.8) (drill 0.4) (layers F.Cu B.Cu) (net 1))
@@
   (via (at 97.028 47.244) (size 0.8) (drill 0.4) (layers F.Cu B.Cu) (net 1))
   (via (at 98.425 48.514) (size 0.8) (drill 0.4) (layers F.Cu B.Cu) (net 1))
-  (via (at 84.328 87.503) (size 0.8) (drill 0.4) (layers F.Cu B.Cu) (net 1))
+  (via (at 83.82 86.2965) (size 0.8) (drill 0.4) (layers F.Cu B.Cu) (net 1))
   (segment (start 88.265 41.275) (end 98.425 41.275) (width 0.65) (layer F.Cu) (net 1))
+  (via (at 75.2475 65.0875) (size 0.8) (drill 0.4) (layers F.Cu B.Cu) (net 1))
+  (via (at 75.311 66.6115) (size 0.8) (drill 0.4) (layers F.Cu B.Cu) (net 1))
+  (via (at 77.978 62.9285) (size 0.8) (drill 0.4) (layers F.Cu B.Cu) (net 1))
+  (via (at 78.0415 63.8175) (size 0.8) (drill 0.4) (layers F.Cu B.Cu) (net 1))
+  (via (at 80.264 61.9125) (size 0.8) (drill 0.4) (layers F.Cu B.Cu) (net 1))
+  (via (at 81.3435 65.024) (size 0.8) (drill 0.4) (layers F.Cu B.Cu) (net 1))
+  (via (at 79.5655 67.183) (size 0.8) (drill 0.4) (layers F.Cu B.Cu) (net 1))
+  (via (at 78.8035 75.7555) (size 0.8) (drill 0.4) (layers F.Cu B.Cu) (net 1))
+  (via (at 78.359 77.089) (size 0.8) (drill 0.4) (layers F.Cu B.Cu) (net 1))
+  (via (at 69.977 80.0735) (size 0.8) (drill 0.4) (layers F.Cu B.Cu) (net 1))
+  (via (at 85.217 81.9785) (size 0.8) (drill 0.4) (layers F.Cu B.Cu) (net 1))
+  (via (at 82.804 82.677) (size 0.8) (drill 0.4) (layers F.Cu B.Cu) (net 1))
+  (via (at 84.201 83.439) (size 0.8) (drill 0.4) (layers F.Cu B.Cu) (net 1))
+  (via (at 82.2325 84.8995) (size 0.8) (drill 0.4) (layers F.Cu B.Cu) (net 1))
+  (via (at 81.8515 87.0585) (size 0.8) (drill 0.4) (layers F.Cu B.Cu) (net 1))
+  (via (at 75.6285 45.593) (size 0.8) (drill 0.4) (layers F.Cu B.Cu) (net 1))
+  (via (at 74.422 46.0375) (size 0.8) (drill 0.4) (layers F.Cu B.Cu) (net 1))
+  (via (at 75.311 48.006) (size 0.8) (drill 0.4) (layers F.Cu B.Cu) (net 1))
+  (via (at 74.2315 49.0855) (size 0.8) (drill 0.4) (layers F.Cu B.Cu) (net 1))
+  (via (at 76.073 50.927) (size 0.8) (drill 0.4) (layers F.Cu B.Cu) (net 1))
+  (via (at 73.66 50.4825) (size 0.8) (drill 0.4) (layers F.Cu B.Cu) (net 1))
+  (via (at 69.5325 45.9105) (size 0.8) (drill 0.4) (layers F.Cu B.Cu) (net 1))
+  (via (at 70.5485 46.6725) (size 0.8) (drill 0.4) (layers F.Cu B.Cu) (net 1))
+  (via (at 70.4215 50.1015) (size 0.8) (drill 0.4) (layers F.Cu B.Cu) (net 1))
+  (via (at 69.5325 51.943) (size 0.8) (drill 0.4) (layers F.Cu B.Cu) (net 1))
+  (via (at 81.2165 41.3385) (size 0.8) (drill 0.4) (layers F.Cu B.Cu) (net 1))
+  (via (at 81.2165 42.418) (size 0.8) (drill 0.4) (layers F.Cu B.Cu) (net 1))
+  (via (at 84.3915 41.529) (size 0.8) (drill 0.4) (layers F.Cu B.Cu) (net 1))
+  (via (at 83.3755 43.2435) (size 0.8) (drill 0.4) (layers F.Cu B.Cu) (net 1))
+  (via (at 85.725 43.434) (size 0.8) (drill 0.4) (layers F.Cu B.Cu) (net 1))
+  (via (at 78.105 56.3245) (size 0.8) (drill 0.4) (layers F.Cu B.Cu) (net 1))
+  (via (at 78.359 57.912) (size 0.8) (drill 0.4) (layers F.Cu B.Cu) (net 1))
+  (via (at 79.248 48.9585) (size 0.8) (drill 0.4) (layers F.Cu B.Cu) (net 1))
   (segment (start 72.771 52.832) (end 75.311 52.832) (width 0.65) (layer F.Cu) (net 2))
   (segment (start 78.994 52.832) (end 82.931 48.895) (width 0.65) (layer F.Cu) (net 2))
@@
   (segment (start 76.2 72.657) (end 76.2 68.199) (width 0.65) (layer F.Cu) (net 4))
   (segment (start 88.265 88.265) (end 98.425 88.265) (width 0.65) (layer F.Cu) (net 4))
-  (segment (start 84.772001 88.428001) (end 84.935002 88.265) (width 0.65) (layer F.Cu) (net 4))
-  (segment (start 83.883999 88.428001) (end 84.772001 88.428001) (width 0.65) (layer F.Cu) (net 4))
-  (segment (start 71.882 88.265) (end 83.720998 88.265) (width 0.65) (layer F.Cu) (net 4))
   (segment (start 84.935002 88.265) (end 88.265 88.265) (width 0.65) (layer F.Cu) (net 4))
+  (segment (start 71.882 88.265) (end 84.935002 88.265) (width 0.65) (layer F.Cu) (net 4))
   (segment (start 74.409 72.657) (end 73.406 73.66) (width 0.65) (layer F.Cu) (net 4))
   (segment (start 76.2 72.657) (end 74.409 72.657) (width 0.65) (layer F.Cu) (net 4))
+  (segment (start 69.977 82.423) (end 69.977 86.36) (width 0.65) (layer F.Cu) (net 4))
   (segment (start 73.406 73.66) (end 73.406 78.994) (width 0.65) (layer F.Cu) (net 4))
-  (segment (start 83.720998 88.265) (end 83.883999 88.428001) (width 0.65) (layer F.Cu) (net 4))
   (segment (start 73.406 78.994) (end 69.977 82.423) (width 0.65) (layer F.Cu) (net 4))
-  (segment (start 69.977 82.423) (end 69.977 86.36) (width 0.65) (layer F.Cu) (net 4))
   (segment (start 69.977 86.36) (end 71.882 88.265) (width 0.65) (layer F.Cu) (net 4))
   (segment (start 78.486 70.485) (end 81.661 67.31) (width 0.65) (layer F.Cu) (net 5))
